Commit message: Robot Sensor:Done

File: src/my_robot/urdf/my_robot.xacro (robot description, xacro)
@@ -8,5 +8,5 @@
   </joint>
   <joint type="continuous" name="left_wheel_hinge">
-    <origin xyz="0 0.125 0" rpy="0 0 0"/>
+    <origin xyz="0 0.15 0" rpy="0 0 0"/>
     <child link="left_wheel"/>
     <parent link="chassis"/>
@@ -16,5 +16,5 @@
   </joint>
   <joint type="continuous" name="right_wheel_hinge">
-    <origin xyz="0 -0.125 0" rpy="0 0 0"/>
+    <origin xyz="0 -0.15 0" rpy="0 0 0"/>
     <child link="right_wheel"/>
     <parent link="chassis"/>
@@ -22,4 +22,16 @@
     <limit effort="10000" velocity="1000"/>
     <dynamics damping="1.0" friction="1.0"/>
+  </joint>
+  <joint name="camera_joint" type="fixed">
+    <origin xyz="0.2 0 0" rpy="0 0 0"/>
+    <child link="camera"/>
+    <parent link="chassis"/>
+    <axis xyz="0 1 0" rpy="0 0 0"/>
+  </joint>
+  <joint name="hokuyo_joint" type="fixed">
+    <origin xyz="0.15 0 0.1" rpy="0 0 0"/>
+    <child link="hokuyo"/>
+    <parent link="chassis"/>
+    <axis xyz="0 1 0" rpy="0 0 0"/>
   </joint>
   <link name='chassis'>
@@ -119,3 +131,67 @@
   </visual>
 </link>
+<link name='camera'>
+  <pose>0 0 0 0 0 0</pose>
+  <inertial>
+    <mass value="0.1"/>
+    <origin xyz="0 0 0" rpy=" 0 0 0"/>
+    <inertia
+        ixx="1e-6" ixy="0" ixz="0"
+        iyy="1e-6" iyz="0"
+        izz="1e-6"
+    />
+    <box_inertia m="0.1" x="0.05" y="0.05" z="0.05" />
+  </inertial>
+  <collision name='collision'>
+    <origin xyz="0 0 0" rpy=" 0 0 0"/>
+    <geometry>
+      <box size="0.05 0.05 0.05"/>
+    </geometry>
+  </collision>
+  <visual name='camera_visual'>
+    <origin xyz="0 0 0" rpy=" 0 0 0"/>
+    <geometry>
+      <box size="0.05 0.05 0.05"/>
+    </geometry>
+    <material name="Cyan">
+      <color rgba="0 1.0 1.0 1.0"/>
+    </material>
+  </visual>
+</link>
+<link name='hokuyo'>
+  <pose>0 0 0 0 0 0</pose>
+  <inertial>
+    <mass value="1e-5"/>
+    <origin xyz="0 0 0" rpy=" 0 0 0"/>
+    <inertia
+        ixx="1e-6" ixy="0" ixz="0"
+        iyy="1e-6" iyz="0"
+        izz="1e-6"
+    />
+  </inertial>
+  <collision name='collision'>
+    <origin xyz="0 0 0" rpy=" 0 0 0"/>
+    <geometry>
+      <box size="0.1 0.1 0.1"/>
+    </geometry>
+  </collision>
+  <visual name='hokuyo_visual'>
+    <origin xyz="0 0 0" rpy=" 0 0 0"/>
+    <geometry>
+      <mesh filename="package://my_robot/meshes/hokuyo.dae"/>
+    </geometry>
+  </visual>
+</link>
+<gazebo reference="left_wheel">
+    <material>Gazebo/Green</material>
+</gazebo>
+<gazebo reference="right_wheel">
+    <material>Gazebo/Green</material>
+</gazebo>
+<gazebo reference="chassis">
+    <material>Gazebo/Blue</material>
+</gazebo>
+<gazebo reference="camera">
+    <material>Gazebo/Red</material>
+</gazebo>
 </robot>

Commit message: map my world

File: src/my_robot/urdf/my_robot.xacro (robot description, xacro)
@@ -2,4 +2,11 @@
 <robot name="my_robot" xmlns:xacro="http://www.ros.org/wiki/xacro">
   <xacro:include filename="$(find my_robot)/urdf/my_robot.gazebo" />
+  <joint name="camera_optical_joint" type="fixed">
+    <origin xyz="0 0 0" rpy="-1.5707 0 -1.5707"/>
+    <parent link="camera"/>
+    <child link="camera_link_optical"/>
+  </joint>
+  <link name="camera_link_optical">
+  </link>
   <link name="robot_footprint"></link>
   <joint name="robot_footprint_joint" type="fixed">
